Commit message: git-svn-id: file:///home/svn/m3meka@218 1168f755-9803-407b-a38c-2651d5e71887

File: branches/iq/meka-ros/meka_common/meka_description/robots/meka.urdf.xacro (robot description, xacro)
@@ -47,5 +47,5 @@
 		  <origin xyz="0 0 0" rpy="0 0 0" />
 		  <geometry name="upper_geom">
-			  <mesh filename="package://${MESH}/T2R3/T2R3_TJ3_chest_waist_neck.dae" />
+			  <mesh filename="package://${MESH}/A2R3/A2R3_T4_Chest.dae" />
 		  </geometry>
 	  </visual>
@@ -53,5 +53,5 @@
 		  <origin xyz="0 0 0" rpy="0.0 0.0 0.0 " />
 		  <geometry name="upper_collision_geom">
-			  <mesh filename="package://${MESH_COLL}/T2R3/T2R3_TJ3_chest_waist_neck.stl" />
+			  <mesh filename="package://${MESH_COLL}/A2R3/A2R3_T4_Chest.stl" />
 		  </geometry>
 	  </collision>
